File: LT8490.kicad_sch (KiCad schematic)
At the start: 122 parts, among them J1 Conn_01x01, J10 Conn_01x01, J11 Conn_01x01, J12 Conn_01x01, J13 Conn_01x01, J14 Conn_01x01, J15 Conn_01x01, J16 Conn_01x01, J17 Conn_01x01, J18 Conn_01x01, J19 Conn_01x01, J2 Conn_01x01, J20 Conn_01x01, J21 Conn_01x01, J22 Conn_01x01, J23 Conn_01x01, J24 Conn_01x01, J25 Conn_01x01, J3 Conn_01x01, J4 Conn_01x01, J5 Conn_01x01, J6 Conn_01x01, J7 Conn_01x01, J8 Conn_01x01, J9 Conn_01x01, Q1 Si7106DN, Q2 Si7106DN, Q3 Si7106DN, Q4 Si7106DN, Q5 BSS84, Q6 MBT2222ADW1T1, U4 LT8490EUKJPBF

Commit message: beefed up LDO3V3
Parts:
- D1, D2: footprint Diode_SMD:D_SOD-123F -> Diode_SMD:D_PowerDI-123
Changed lines of the file:
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@@
       (effects (font (size 1.27 1.27)) (justify right))
     )
-    (property "Footprint" "Diode_SMD:D_SOD-123F" (id 2) (at 132.08 50.8 0)
+    (property "Footprint" "Diode_SMD:D_PowerDI-123" (id 2) (at 132.08 50.8 0)
       (effects (font (size 1.27 1.27)) hide)
     )
@@
       (effects (font (size 1.27 1.27)) (justify right))
     )
-    (property "Footprint" "Diode_SMD:D_SOD-123F" (id 2) (at 113.03 50.8 0)
+    (property "Footprint" "Diode_SMD:D_PowerDI-123" (id 2) (at 113.03 50.8 0)
       (effects (font (size 1.27 1.27)) hide)
     )
@@
     )
     (path "/735821d5-c933-409c-b96d-1d60d9085727"
-      (reference "D1") (unit 1) (value "MBR1020VL") (footprint "Diode_SMD:D_SOD-123F")
+      (reference "D1") (unit 1) (value "MBR1020VL") (footprint "Diode_SMD:D_PowerDI-123")
     )
     (path "/528ec391-38c0-4c96-9975-7dacb1e30217"
-      (reference "D2") (unit 1) (value "MBR1020VL") (footprint "Diode_SMD:D_SOD-123F")
+      (reference "D2") (unit 1) (value "MBR1020VL") (footprint "Diode_SMD:D_PowerDI-123")
     )
     (path "/3b48b997-b2e1-4d81-af37-fb5bf851b4f4"
